Commit message: Adding _joint to joints (moer PR2 like)

File: albany_robots/albany_common/launch/ROSalyn.urdf (robot description, URDF)
Before this commit: robot ROSalyn, 6 links, 5 joints
Joints:
- removed joint head_pan
- removed joint head_tilt
- removed joint laser
- added joint head_pan_joint: type revolute, parent column_link, child pan_link, origin xyz=0.0762 0 0, axis 0 0 1.0, limit lower=-1.57 upper=1.57 effort=30 velocity=1.0
- added joint head_tilt_joint: type revolute, parent pan_link, child tilt_link, origin xyz=.0381 0 .0381 , axis 0 1.0 0, limit lower=-1.57 upper=1.57 effort=30 velocity=1.0
- added joint laser_joint: type fixed, parent base_link, child base_laser, origin xyz=0 0 0.165
